File: DingoPDM/BTS700n_1EPP.kicad_sch (KiCad schematic)
At the start: 13 parts, among them U8 BTS700n-1EPP

Commit message: Modified PCB for 10ch PDM board
I modified the original dingoPDM for 10 channels. The board has been manufactured, tested and works but after mounting I decided that it doesn't suit my needs for the current build. I may develop it further in the future, make it pretty etc but for now I am marking this project as stale.
Parts:
- D8: footprint dingoPDM:DO-214AC -> digikey-footprints:DO-214AC
- U8: footprint dingoPDM:TDSO-14 -> Profet:TDSO-14
Changed lines of the file:
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@@
 			)
 		)
-		(property "Footprint" "dingoPDM:TDSO-14"
+		(property "Footprint" "Profet:TDSO-14"
 			(at 121.92 82.55 0)
 			(effects
@@
 			)
 		)
-		(property "Footprint" "dingoPDM:DO-214AC"
+		(property "Footprint" "digikey-footprints:DO-214AC"
 			(at 170.18 104.14 0)
 			(effects
