File: DingoPDM/MCU.kicad_sch (KiCad schematic)
At the start: 29 parts, among them J4 TC, SW1 BOOT, U3 PCA82C250, U4 STM32F446RETx, Y1 8mHz

Commit message: Modified PCB for 10ch PDM board
I modified the original dingoPDM for 10 channels. The board has been manufactured, tested and works but after mounting I decided that it doesn't suit my needs for the current build. I may develop it further in the future, make it pretty etc but for now I am marking this project as stale.
Parts:
- removed TP10: E3, TestPoint:TestPoint_Keystone_5000-5004_Miniature, symbol Connector:TestPoint
- removed TP2: CAN_T, TestPoint:TestPoint_Keystone_5000-5004_Miniature, symbol Connector:TestPoint
- removed TP3: CAN_R, TestPoint:TestPoint_Keystone_5000-5004_Miniature, symbol Connector:TestPoint
- removed TP8: E1, TestPoint:TestPoint_Keystone_5000-5004_Miniature, symbol Connector:TestPoint
- removed TP9: E2, TestPoint:TestPoint_Keystone_5000-5004_Miniature, symbol Connector:TestPoint
Connections:
- net PF_IN7: now also U4.41 (PA8); no longer U4.23 (PA7)
- net PF_DEN9_10: now reaches U4.34 (PB13)
- net PF_DSEL9_10: now reaches U4.50 (PA15)
- net PF_IN9: now reaches U4.56 (PB4)
- net PF_IN10: now reaches U4.57 (PB5)
- net PF1_IS: no longer names the net of U4.14 (PA0)
- net PF2_IS renamed PF_IS9_10
- net PF_DEN1 renamed PF_DEN1_2
- net PF_DEN2 renamed PF_DSEL1_2
- net USB_DM: no longer names the net of U4.44 (PA11)
- net USB_DP: no longer names the net of U4.45 (PA12)
- net USB_VBUS: no longer names the net of U4.42 (PA9)
- new net PF_IS1_2: U4.23 (PA7)
- no-connect marks 8 -> 3
Other:
- note added: "MODIFIED"
