File: DingoPDM/Power.kicad_sch (KiCad schematic)
At the start: 18 parts, among them U1 VXO7805-500-M, U14 OKI-78SR-5_1.5-W36H-C, U15 TSR_1-2450, U2 LD1117S33CTR

Commit message: Modified PCB for 10ch PDM board
I modified the original dingoPDM for 10 channels. The board has been manufactured, tested and works but after mounting I decided that it doesn't suit my needs for the current build. I may develop it further in the future, make it pretty etc but for now I am marking this project as stale.
Parts:
- removed TP1: GND, TestPoint:TestPoint_Keystone_5000-5004_Miniature, symbol Connector:TestPoint
- U1: LCSC C5137464 -> (none)
- U14: footprint dingoPDM:Converter_DCDC_Murata_OKI-78SR_Horizontal -> Converter_DCDC:Converter_DCDC_Murata_OKI-78SR_Horizontal; Digi-Key_PN 811-2692-ND -> (none); LCSC C266374 -> (none)
- U15: footprint dingoPDM:Converter_DCDC_TRACO_TSR-1_THT -> Converter_DCDC:Converter_DCDC_TRACO_TSR-1_THT; Digi-Key_PN 1951-2747-ND -> (none); LCSC C6886877 -> (none)
Changed lines of the file:
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@@
 			)
 		)
-		(property "LCSC" "C5137464"
+		(property "LCSC" ""
 			(at 99.06 34.29 0)
 			(effects
@@
 	)
 	(symbol
-		(lib_id "Connector:TestPoint")
-		(at 69.215 53.34 0)
-		(unit 1)
-		(exclude_from_sim no)
-		(in_bom yes)
-		(on_board yes)
-		(dnp no)
-		(property "Reference" "TP1"
-			(at 70.6882 50.3428 0)
-			(effects
-				(font
-					(size 1.27 1.27)
-				)
-				(justify left)
-			)
-		)
-		(property "Value" "GND"
-			(at 70.6882 52.6542 0)
-			(effects
-				(font
-					(size 1.27 1.27)
-				)
-				(justify left)
-			)
-		)
-		(property "Footprint" "TestPoint:TestPoint_Keystone_5000-5004_Miniature"
-			(at 74.295 53.34 0)
-			(effects
-				(font
-					(size 1.27 1.27)
-				)
-				(hide yes)
-			)
-		)
-		(property "Datasheet" ""
-			(at 74.295 53.34 0)
-			(effects
-				(font
-					(size 1.27 1.27)
-				)
-				(hide yes)
-			)
-		)
-		(property "Description" ""
-			(at 69.215 53.34 0)
-			(effects
-				(font
-					(size 1.27 1.27)
-				)
-				(hide yes)
-			)
-		)
-		(property "LCSC" ""
-			(at 69.215 53.34 0)
-			(effects
-				(font
-					(size 1.27 1.27)
-				)
-				(hide yes)
-			)
-		)
-		(pin "1"
-		)
-		(instances
-			(project "DingoPDM"
-				(path "/8948e307-9174-4227-9c28-3ff885e6e83d/00000000-0000-0000-0000-00005f5cf2eb"
-					(reference "TP1")
-					(unit 1)
-				)
-			)
-		)
-	)
-	(symbol
-		(lib_id "power:GND")
-		(at 69.215 53.34 0)
-		(unit 1)
-		(exclude_from_sim no)
-		(in_bom yes)
-		(on_board yes)
-		(dnp no)
-		(property "Reference" "#PWR08"
-			(at 69.215 59.69 0)
-			(effects
-				(font
-					(size 1.27 1.27)
-				)
-				(hide yes)
-			)
-		)
-		(property "Value" "GND"
-			(at 69.342 57.7342 0)
-			(effects
-				(font
-					(size 1.27 1.27)
-				)
-			)
-		)
-		(property "Footprint" ""
-			(at 69.215 53.34 0)
-			(effects
-				(font
-					(size 1.27 1.27)
-				)
-				(hide yes)
-			)
-		)
-		(property "Datasheet" ""
-			(at 69.215 53.34 0)
-			(effects
-				(font
-					(size 1.27 1.27)
-				)
-				(hide yes)
-			)
-		)
-		(property "Description" ""
-			(at 69.215 53.34 0)
-			(effects
-				(font
-					(size 1.27 1.27)
-				)
-				(hide yes)
-			)
-		)
-		(pin "1"
-		)
-		(instances
-			(project "DingoPDM"
-				(path "/8948e307-9174-4227-9c28-3ff885e6e83d/00000000-0000-0000-0000-00005f5cf2eb"
-					(reference "#PWR08")
-					(unit 1)
-				)
-			)
-		)
-	)
-	(symbol
 		(lib_id "Device:LED_Small")
 		(at 212.09 46.355 90)
@@
 			)
 		)
-		(property "Footprint" "dingoPDM:Converter_DCDC_Murata_OKI-78SR_Horizontal"
+		(property "Footprint" "Converter_DCDC:Converter_DCDC_Murata_OKI-78SR_Horizontal"
 			(at 39.37 78.74 0)
 			(effects
@@
 		)
 		(property "Description" "1.5A Step-Down DC/DC-Regulator, 7-36V input, 5V fixed Output Voltage, LM78xx replacement, -40°C to +85°C, OKI-78SR_Horizontal"
-			(at 38.1 72.39 0)
-			(effects
-				(font
-					(size 1.27 1.27)
-				)
-				(hide yes)
-			)
-		)
-		(property "Digi-Key_PN" "811-2692-ND"
-			(at 38.1 72.39 0)
-			(effects
-				(font
-					(size 1.27 1.27)
-				)
-				(hide yes)
-			)
-		)
-		(property "LCSC" "C266374"
 			(at 38.1 72.39 0)
 			(effects
@@
 			)
 		)
-		(property "Footprint" "dingoPDM:Converter_DCDC_TRACO_TSR-1_THT"
+		(property "Footprint" "Converter_DCDC:Converter_DCDC_TRACO_TSR-1_THT"
 			(at 38.1 114.3 0)
 			(effects
@@
 			(at 38.1 110.49 0)
 			(effects
-				(font
-					(size 1.27 1.27)
-				)
-				(hide yes)
-			)
-		)
-		(property "Digi-Key_PN" "1951-2747-ND"
-			(at 38.1 110.49 0)
-			(effects
-				(font
-					(size 1.27 1.27)
-				)
-				(hide yes)
-			)
-		)
-		(property "LCSC" "C6886877"
-			(at 38.1 110.49 0)
-			(effects
